Commit message: Updated right_wheel_joint axis to fix translation in teleop

File: src/igvc_description/urdf/model.urdf.xacro (robot description, xacro)
@@ -680,5 +680,5 @@
     <parent link="part_1"/>
     <child link="part_34"/>
-    <axis xyz="0 0 1"/>
+    <axis xyz="0 0 -1"/>
     <limit effort="10" velocity="10" lower="-3.141592653589793" upper="3.141592653589793"/>
   </joint>
