Commit message: Test Day 4 Changes

File: src/igvc_description/urdf/robot.urdf.xacro (robot description, xacro)
@@ -7,5 +7,5 @@
     <joint name="base_joint" type="fixed">
         <parent link="base_link"/>
-        <origin rpy="0 0 0" xyz="0 0 0.01"/>
+        <origin rpy="0 0 ${-pi/2}" xyz="0 0 0.01"/>
         <child link="part_1"/>
         <axis xyz="0 0 1"/>

File: src/igvc_description/urdf/sensor/lidar.urdf.xacro (robot description, xacro)
@@ -4,5 +4,5 @@
         <parent link="base_link"/>
         <child link="laser_frame"/>
-        <origin xyz="-0.05 0.605 0.50" rpy="0 0 ${-pi/2}"/>
+        <origin xyz="0.605 0 0.50" rpy="0 0 ${pi}"/>
     </joint>
     <link name="laser_frame">

Commit message: measurinator 8000 dummy

File: src/igvc_description/urdf/robot.urdf.xacro (robot description, xacro)
@@ -1,28 +1,10 @@
 <?xml version="1.0" ?>
 <robot xmlns:xacro="http://www.ros.org/wiki/xacro" name="igvc_robot">
-    <xacro:arg name="prefix" default="" />
-    <xacro:arg name="use_mock_hardware" default="false" />
-    <link name="base_footprint"/>
     <link name="base_link"/>
-    <joint name="base_joint" type="fixed">
+    <link name="zed_camera_link"/>
+    <joint name="camera_joint" type="fixed">
         <parent link="base_link"/>
-        <origin rpy="0 0 0" xyz="0 0 0.01"/>
-        <child link="part_1"/>
-        <axis xyz="0 0 1"/>
+        <origin rpy="0 0 0" xyz="0 0 1.0795"/>
+        <child link="zed_camera_link"/>
     </joint>
-    <joint name="footprint_joint" type="fixed">
-        <parent link="base_link"/>
-        <origin rpy="0 0 0" xyz="0 0 0.01"/>
-        <child link="base_footprint"/>
-        <axis xyz="0 0 1"/>
-    </joint>
-    <xacro:include filename="$(find igvc_description)/urdf/model.urdf.xacro"/>
-    <xacro:include filename="$(find igvc_description)/urdf/sensors.urdf.xacro"/>
-    <xacro:include filename="$(find igvc_description)/control/bot.ros2_control.xacro" />
-    <xacro:bot_ros2_control name="IGVC_Bot" prefix="$(arg prefix)" use_mock_hardware="$(arg use_mock_hardware)"/>
-    <gazebo>
-        <plugin filename="gz_ros2_control-system" name="gz_ros2_control::GazeboSimROS2ControlPlugin">
-        <parameters>$(find igvc_hardware)/config/bot_controllers.yaml</parameters>
-        </plugin>
-    </gazebo>
 </robot>
